File: LCB-CDB-01/Connector_Control_Board.kicad_sch (KiCad schematic)
At the start: 1 part, among them J402 LCB_connector_top

Commit message: bump version to 1.1.0
Other:
- title: LCB-CBD-001: Dock -> LCB-CBD-01: Dock
Changed lines of the file:
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@@
   (paper "A4")
   (title_block
-    (title "LCB-CBD-001: Dock")
-    (date "2022-08-12")
-    (rev "0.1")
+    (title "LCB-CBD-01: Dock")
+    (date "2023-04-13")
+    (rev "1.1.0")
     (company "PADERBORN UNIVERSITY DEPARTMENT OF POWER ELECTRONICS AND ELECTRICAL DRIVES")
   )

Commit message: update symbols without simulation models
Parts:
- J402: Mfr. No ERF5-075-05.0-L-DV-TR -> (none); Mouser No 200-ERF507505.0LDVTR -> (none)
Other:
- title: LCB-CBD-01: Dock -> LCB-CDB-01: Dock Board
Changed lines of the file:
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@@
 	(paper "A4")
 	(title_block
-		(title "LCB-CBD-01: Dock")
-		(date "2024-06-25")
+		(title "LCB-CDB-01: Dock Board")
+		(date "2024-07-16")
 		(rev "1.2.0")
 		(company "PADERBORN UNIVERSITY DEPARTMENT OF POWER ELECTRONICS AND ELECTRICAL DRIVES")
@@
 		(at 19.05 38.1 0)
 		(unit 1)
-		(exclude_from_sim no)
+		(exclude_from_sim yes)
 		(in_bom yes)
 		(on_board yes)
@@
 		(at 247.65 113.03 0)
 		(unit 4)
-		(exclude_from_sim no)
+		(exclude_from_sim yes)
 		(in_bom yes)
 		(on_board yes)
@@
 			)
 		)
-		(property "Mouser No" "200-ERF507505.0LDVTR"
-			(at 285.75 100.33 0)
-			(effects
-				(font
-					(size 1.27 1.27)
-				)
-				(hide yes)
-			)
-		)
-		(property "Mfr. No" "ERF5-075-05.0-L-DV-TR"
-			(at 287.02 102.87 0)
-			(effects
-				(font
-					(size 1.27 1.27)
-				)
-				(hide yes)
-			)
-		)
 		(property "mouser#" "200-ERF507505.0LDVTR"
 			(at 285.75 100.33 0)
@@
 		(at 19.05 26.67 0)
 		(unit 1)
-		(exclude_from_sim no)
+		(exclude_from_sim yes)
 		(in_bom yes)
 		(on_board yes)
@@
 		(at 180.34 113.03 0)
 		(unit 3)
-		(exclude_from_sim no)
+		(exclude_from_sim yes)
 		(in_bom yes)
 		(on_board yes)
@@
 			)
 		)
-		(property "Mouser No" "200-ERF507505.0LDVTR"
-			(at 218.44 100.33 0)
-			(effects
-				(font
-					(size 1.27 1.27)
-				)
-				(hide yes)
-			)
-		)
-		(property "Mfr. No" "ERF5-075-05.0-L-DV-TR"
-			(at 219.71 102.87 0)
-			(effects
-				(font
-					(size 1.27 1.27)
-				)
-				(hide yes)
-			)
-		)
 		(property "mouser#" "200-ERF507505.0LDVTR"
 			(at 218.44 100.33 0)
@@
 		(at 53.34 113.03 0)
 		(unit 1)
-		(exclude_from_sim no)
+		(exclude_from_sim yes)
 		(in_bom yes)
 		(on_board yes)
@@
 			)
 		)
-		(property "Mouser No" "200-ERF507505.0LDVTR"
-			(at 91.44 100.33 0)
-			(effects
-				(font
-					(size 1.27 1.27)
-				)
-				(hide yes)
-			)
-		)
-		(property "Mfr. No" "ERF5-075-05.0-L-DV-TR"
-			(at 92.71 102.87 0)
-			(effects
-				(font
-					(size 1.27 1.27)
-				)
-				(hide yes)
-			)
-		)
 		(property "mouser#" "200-ERF507505.0LDVTR"
 			(at 91.44 100.33 0)
@@
 		(at 118.11 111.76 0)
 		(unit 2)
-		(exclude_from_sim no)
+		(exclude_from_sim yes)
 		(in_bom yes)
 		(on_board yes)
@@
 			(effects
 				(font
-					(size 1.27 1.27)
-				)
-				(hide yes)
-			)
-		)
-		(property "Mouser No" "200-ERF507505.0LDVTR"
-			(at 156.21 99.06 0)
-			(effects
-				(font
-					(size 1.27 1.27)
-				)
-				(hide yes)
-			)
-		)
-		(property "Mfr. No" "ERF5-075-05.0-L-DV-TR"
-			(at 157.48 101.6 0)
-			(effects
-				(font
